File: board/smart-wipers-board/smart-wipers-board.kicad_pcb (KiCad board)
At the start: 2 copper layers, 45 x 51 mm, 38 parts, among them J1 X1, J10 XCAN, J7 X2, J8 XC1, J9 XC2, U1 STM32F105R8Tx, U2 SN65HVD232, U3 SN65HVD232, U4 ST1S10PHR, Y1 8Mhz

Commit message: WIP Board design
Parts:
- C14, C15: value 20pF -> 15pF
- J10: footprint Connector_PinHeader_2.54mm:PinHeader_2x08_P2.54mm_Vertical -> Connector:OBD; moved to F.Cu
- L1: footprint Inductor_SMD:L_6.3x6.3_H3 -> Inductor_SMD:L_7.3x7.3_H3.5
- R1, R2: moved to F.Cu
- Y1: footprint SparkFun-FreqCtrl:HC49US -> Crystal:Crystal_SMD_5032-2Pin_5.0x3.2mm_HandSoldering; moved to B.Cu
- moved C3 25.0 mm to (42.2, 31.1), turned to 270 degrees
- moved C15 21.4 mm to (44.5, 31.1)
- moved R1 17.6 mm to (23.0, 13.6), turned to 180 degrees
- moved C14 16.9 mm to (42.4, 14.9)
- moved Y1 16.2 mm to (42.4, 22.6)
- moved J10 6.68 mm to (48.6, 48.4), turned to 0 degrees
- moved R2 3.04 mm to (17.9, 13.6), turned to 180 degrees
- moved L1 0.98 mm to (20.0, 28.0), turned to 0 degrees
- moved C16 0.32 mm to (50.0, 16.4)
Connections:
- net Net-(R1-Pad2) renamed /FB
- J10 pad 11: (no net) -> CAN_MSL
- J10 pad 3: (no net) -> CAN_MSH
- J10 pad 4: (no net) -> CAN_GND
- J10 pad 5: CAN_MSH -> CAN_GND
- J10 pad 6: CAN_MSL -> (no net)
- J10 pad 7: CAN_GND -> (no net)
- J10 pad 9: CAN_GND -> (no net)
- J9 pad 1: CAN_LSH -> CAN_GND
- J9 pad 2: CAN_GND -> CAN_LSH
- J9 pad 6: CAN_MSH -> CAN_MSL
- J9 pad 7: CAN_MSL -> CAN_MSH
Routing:
- net CAN_GND: track 3.54 -> 103.6 mm
- net /FB: track 29.2 -> 4.89 mm, vias 2 -> 0
- net OSC_IN: track 6.87 -> 19.6 mm, vias 0 -> 1
- net VDD: track 114.4 -> 123.1 mm
- net RESET: track 10.6 -> 16.7 mm
- net GNDREF: track 89.0 -> 94.0 mm, vias 4 -> 3
- net +12V: track 51.2 -> 55.5 mm
- net Net-(L1-Pad1): track 3.15 -> 7.45 mm
- net CAN_MSL: track 18.6 -> 22.8 mm
- net CAN_MSH: track 19.9 -> 16.9 mm
- net CAN_LSH: track 13.6 -> 11.6 mm
- net LSCAN_TX: track 7.10 -> 8.90 mm, vias 2 -> 0
- net CAN_12v: track 13.9 -> 12.2 mm
- net Net-(C15-Pad1): track 15.0 -> 13.7 mm
- net UART_TX: track 28.5 -> 29.3 mm
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- removed copper zone on B.Cu, net CAN_GND
Other:
- board text added: "CarMod Universal Board v0.1"
- board text added: "JLCJLCJLCJLC"

Commit message: WIP Board v0.2 design
Parts:
- added C18: 1uF, Capacitor_SMD:C_1206_3216Metric_Pad1.33x1.80mm_HandSolder, F.Cu at (17.8, 58.2)
- added C19: 10nF, Capacitor_SMD:C_1206_3216Metric_Pad1.33x1.80mm_HandSolder, F.Cu at (22.6, 52.2)
- added C20: 2.2uF, Capacitor_SMD:C_1206_3216Metric_Pad1.33x1.80mm_HandSolder, F.Cu at (17.8, 46.1)
- added C21: 100uF 6.3V, Capacitor_SMD:CP_Elec_6.3x5.4, B.Cu at (49.5, 28.2)
- added R8: 15, Resistor_SMD:R_1206_3216Metric_Pad1.30x1.75mm_HandSolder, B.Cu at (26.2, 23.1)
- added U5: LP2985-5.0, Package_TO_SOT_SMD:SOT-23-5, F.Cu at (19.6, 52.5)
- U3: value SN65HVD232 -> MCP2551-I-SN
- moved C16 30.9 mm to (19.2, 16.8)
- moved C5 15.2 mm to (47.4, 31.0)
- moved C7 15.1 mm to (47.2, 15.7)
- moved C17 4.98 mm to (20.2, 28.2), turned to 270 degrees
- moved C1 4.91 mm to (23.2, 15.5)
- moved U4 0.71 mm to (18.5, 19.5)
- moved R1 0.64 mm to (23.0, 14.2)
- moved R2 0.62 mm to (17.9, 14.2)
- moved C2 0.59 mm to (25.4, 30.4)
- moved C14 0.58 mm to (42.4, 15.5)
- moved C13 0.56 mm to (35.1, 15.5)
- moved C4 0.56 mm to (39.9, 15.5)
- moved C9 0.56 mm to (37.5, 15.5)
- moved R6 0.56 mm to (32.6, 15.5)
- moved R5 0.55 mm to (39.8, 30.5)
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Connections:
- C5 pad 1: VDD -> +5V
- J1 pad 2: +12V -> +5V
- J1 pad 3: (no net) -> GNDREF
- J1 pad 4: (no net) -> +12V
- J8 pad 2: CAN_12v -> CAN_GND
- J8 pad 3: CAN_GND -> CAN_12v
- J8 pad 4: CAN_GND -> CAN_5v
- U1 pad 23: (no net) -> LS_CONTROL
- U3 pad 1: LSCAN_RX -> LSCAN_TX
- U3 pad 3: VDD -> +5V
- U3 pad 4: LSCAN_TX -> LSCAN_RX
- U3 pad 8: (no net) -> LS_CONTROL
Routing:
- net +5V: track 0.00 -> 60.0 mm, vias 0 -> 3
- net +12V: track 55.5 -> 19.1 mm, vias 1 -> 2
- net LS_CONTROL: track 0.00 -> 35.6 mm, vias 0 -> 1
- net VDD: track 123.1 -> 108.2 mm
- net CAN_5v: track 0.00 -> 10.9 mm
- net CAN_12v: track 12.2 -> 18.6 mm
- net UART_RX: track 28.0 -> 31.7 mm
- net LSCAN_TX: track 8.90 -> 5.98 mm
- net Net-(C19-Pad1): track 0.00 -> 2.39 mm
- net CAN_GND: track 103.6 -> 105.9 mm
- net BOOT0: track 2.27 -> 4.43 mm
- net GNDREF: track 94.0 -> 96.0 mm, vias 3 -> 5
- net UART_TX: track 29.3 -> 31.2 mm
- net Net-(D3-Pad2): track 1.84 -> 0.80 mm
- net OSC_IN: track 19.6 -> 18.8 mm
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Other:
- board size 45 x 51 mm -> 43 x 49 mm
- board text added: "+5V"
- board text added: "CarMod Universal Board v0.2"
- board text removed: "CarMod Universal Board v0.1"

Commit message: WIP board v0.2 design
Parts:
- moved J10 0.30 mm to (48.5, 48.1)
Connections:
- J8 pad 2: CAN_GND -> CAN_5v
- J8 pad 3: CAN_12v -> CAN_GND
- J8 pad 4: CAN_5v -> CAN_12v
Routing:
- net CAN_GND: track 105.9 -> 111.7 mm
- net CAN_12v: track 18.6 -> 14.1 mm
- net CAN_5v: track 10.9 -> 8.07 mm

Commit message: Board fixes
Parts:
- J10: footprint Connector:OBD -> SparkFun-Connectors:OBDII
- moved J10 14.6 mm to (34.4, 51.6), turned to 180 degrees
- moved U5 1.11 mm to (18.6, 51.9)
- moved C19 0.31 mm to (22.7, 51.9)
- moved C20 0.18 mm to (17.6, 46.1)
- moved C18 0.18 mm to (17.6, 58.2)
Routing:
- net CAN_LSH: track 12.0 -> 49.0 mm
- net CAN_12v: track 14.1 -> 43.6 mm
- net CAN_GND: track 111.7 -> 94.1 mm
- net CAN_MSH: track 16.8 -> 27.8 mm
- net CAN_MSL: track 22.6 -> 30.2 mm
- net CAN_5v: track 8.07 -> 7.02 mm
- net Net-(C19-Pad1): track 2.39 -> 3.34 mm
